File: T48_TSOP_NOR_Adapter_1-1.kicad_pcb (KiCad board)
At the start: 2 copper layers, 55.9 x 101.6 mm, 25 parts, among them J1 T48_ISP, J2 T48_ISP, P2 27C322, SW1 SW_SPDT, SW2 SW_SPDT, U1 ATtiny25?

Commit message: Add files via upload
Other:
- board text added: "P18/GND/P29"
Changed lines of the file:
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@@
 		)
 	)
-	(gr_text "P29/GND/P18"
-		(at 152.4 116.967 -0)
+	(gr_text "P18/GND/P29"
+		(at 152.4 116.967 0)
 		(layer "B.SilkS")
 		(effects

Commit message: Add files via upload
Parts:
- added TP12: TPB1,27, Bucketmouse:TestPoint_THTPad_D1.5mm_Drill0.7mm, F.Cu at (127.0, 47.0)
- added TP13: TPB1,27, Bucketmouse:TestPoint_THTPad_D1.5mm_Drill0.7mm, F.Cu at (142.2, 47.0)
- added TP14: TPB1,27, Bucketmouse:TestPoint_THTPad_D1.5mm_Drill0.7mm, F.Cu at (139.7, 47.0)
- added TP15: TPB1,27, Bucketmouse:TestPoint_THTPad_D1.5mm_Drill0.7mm, F.Cu at (137.2, 47.0)
- moved TP5 10.2 mm to (129.5, 47.0)
- moved TP7 5.08 mm to (134.6, 47.0)
- moved TP6 2.54 mm to (132.1, 47.0)
Connections:
- net /A0 renamed /ISP3
- net /A1 renamed /ISP6
- net /A10 renamed /ZIF12
- net /A11 renamed /ZIF11
- net /A12 renamed /ZIF10
- net /A13 renamed /ZIF9
- net /A14 renamed /ZIF7
- net /A15 renamed /ZIF6
- net /A16 renamed /ZIF30
- net /A17 renamed /ZIF17
- net /A18 renamed /ZIF16
- net /A19 renamed /ZIF5
- net /A2 renamed /ISP8
- net /A3 renamed /ISP9
- net /A4 renamed /ISP10
- net /A5 renamed /ISP11
- net /A6 renamed /ISP13
- net /A7 renamed /ZIF15
- net /A8 renamed /ZIF14
- net /A9 renamed /ZIF13
- net /D0 renamed /ZIF28
- net /D1 renamed /ZIF27
- net /D10 renamed /ZIF20
- net /D11 renamed /ZIF36
- net /D12 renamed /ZIF35
- net /D13 renamed /ZIF34
- net /D14 renamed /ZIF33
- net /D15 renamed /ZIF32
- net /D2 renamed /ZIF21
- net /D3 renamed /ZIF26
- net /D4 renamed /ZIF25
- net /D5 renamed /ZIF24
- net /D6 renamed /ZIF23
- net /D7 renamed /ZIF22
- net /D8 renamed /ZIF1
- net /D9 renamed /ZIF19
- net /NC renamed /ZIF8
- net /NC10 renamed /ZIF2
- net /NC13 renamed /ZIF40
- net /NC14 renamed /ZIF39
- net /R/~{B} renamed /ZIF38
- net /VCC37 renamed /ZIF37
- net /VSS18 renamed /ZIF18
- net /VSS29 renamed /ZIF29
- net /~{BYTE} renamed /ZIF31
- net /~{CE} renamed /ISP7
- net /~{OE} renamed /ISP5
- net /~{RP} renamed /ZIF4
- net /~{WE} renamed /ZIF3
Routing:
- net /ZIF38: track 2.54 -> 55.0 mm, vias 0 -> 2
- net /ZIF2: track 2.54 -> 44.8 mm, vias 0 -> 2
- net /ZIF39: track 2.54 -> 43.3 mm
- net /ZIF40: track 2.54 -> 39.7 mm
- net /ZIF3: track 81.6 -> 89.3 mm, vias 1 -> 2
- net /ZIF1: track 71.7 -> 73.5 mm
- net /ZIF31: track 146.0 -> 147.8 mm, vias 4 -> 5
- net /ZIF4: track 86.1 -> 87.2 mm
Other:
- board text added: "3"
- board text added: "31"
- board text added: "38"
- board text added: "39"
- board text added: "4"
- board text added: "<"
- board text added: "ZIF PINS"
