File: T48_TSOP_NOR_Adapter_1-1.kicad_sch (KiCad schematic)
At the start: 21 parts, among them J1 T48_ISP, J2 T48_ISP, P2 27C322, SW1 SW_SPDT, SW2 SW_SPDT, U1 ATtiny25?

Commit message: Add files via upload
Parts:
- added TP12, TP13, TP14, TP15: TPB1,27, Bucketmouse:TestPoint_THTPad_D1.5mm_Drill0.7mm, symbol Connector:TestPoint
Connections:
- net A0 renamed ISP3
- net A1 renamed ISP6
- net A10 renamed ZIF12
- net A11 renamed ZIF11
- net A12 renamed ZIF10
- net A13 renamed ZIF9
- net A14 renamed ZIF7
- net A15 renamed ZIF6
- net A16 renamed ZIF30
- net A17 renamed ZIF17
- net A18 renamed ZIF16
- net A19 renamed ZIF5
- net A2 renamed ISP8
- net A3 renamed ISP9
- net A4 renamed ISP10
- net A5 renamed ISP11
- net A6 renamed ISP13
- net A7 renamed ZIF15
- net A8 renamed ZIF14
- net A9 renamed ZIF13
- net D0 renamed ZIF28
- net D1 renamed ZIF27
- net D10 renamed ZIF20
- net D11 renamed ZIF36
- net D12 renamed ZIF35
- net D13 renamed ZIF34
- net D14 renamed ZIF33
- net D15 renamed ZIF32
- net D2 renamed ZIF21
- net D3 renamed ZIF26
- net D4 renamed ZIF25
- net D5 renamed ZIF24
- net D6 renamed ZIF23
- net D7 renamed ZIF22
- net D8 renamed ZIF1
- net D9 renamed ZIF19
- net NC renamed ZIF8
- net NC10 renamed ZIF2
- net ZIF2: now also TP12.1
- net NC13 renamed ZIF40
- net ZIF40: now also TP13.1
- net NC14 renamed ZIF39
- net ZIF39: now also TP14.1
- net R/~{B} renamed ZIF38
- net ZIF38: now also TP15.1
- net VCC37 renamed ZIF37
- net VSS18 renamed ZIF18
- net VSS29 renamed ZIF29
- net ~{BYTE} renamed ZIF31
- net ~{CE} renamed ISP7
- net ~{OE} renamed ISP5
- net ~{RP} renamed ZIF4
- net ~{WE} renamed ZIF3
Other:
- note added: "29F160 NC Pins"
- note added: "29F160 Pins:"
- note added: "NC10"
- note added: "NC13"
- note added: "NC14"
- note added: "NC15"
- note added: "~{BYTE}"
- note added: "~{RP}"
- note added: "~{WE}"
- moved on the sheet: C1, J1, J2, R1, TP1, TP10, TP11, TP2, TP3, TP5, TP6, TP7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
